File: 03_Boards/03_DriverRGB_v1/04_Board.kicad_pcb (KiCad board)
At the start: 2 copper layers, 42.7 x 37.8 mm, 24 parts, among them J1 PJ-102A, J2 LED_OUT, J3 PROG INTERFACE, Q1 BUK9214-30A, Q2 BUK9214-30A, Q3 BUK9214-30A, Q4 BUK9214-30A, U1 ESP-12S, U2 BD33FC0FP

Commit message: PCB
Changed lines of the file:
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@@
   (segment (start 110.998 85.852) (end 109.786 87.064) (width 0.5) (layer "B.Cu") (net 14))
   (segment (start 105.348 87.064) (end 103.948 85.664) (width 0.5) (layer "B.Cu") (net 14))
-  (segment (start 108.028 71.374) (end 110.528 71.374) (width 0.5) (layer "F.Cu") (net 16))
+  (segment (start 108.028 71.374) (end 108.028 71.833) (width 0.5) (layer "F.Cu") (net 16))
   (segment (start 108.458 80.772) (end 110.998 83.312) (width 0.5) (layer "F.Cu") (net 16))
-  (segment (start 110.528 72.674) (end 111.73805 72.674) (width 0.5) (layer "F.Cu") (net 16))
   (segment (start 113.538 74.47395) (end 113.538 80.772) (width 0.5) (layer "F.Cu") (net 16))
-  (segment (start 105.918 72.595) (end 106.807 72.595) (width 0.5) (layer "F.Cu") (net 16))
-  (segment (start 111.73805 72.674) (end 113.538 74.47395) (width 0.5) (layer "F.Cu") (net 16))
+  (segment (start 107.3386 72.595) (end 108.028 71.9056) (width 0.5) (layer "F.Cu") (net 16))
+  (segment (start 105.918 72.595) (end 107.3386 72.595) (width 0.5) (layer "F.Cu") (net 16))
+  (segment (start 108.028 71.9056) (end 108.028 71.374) (width 0.5) (layer "F.Cu") (net 16))
+  (segment (start 113.538 80.772) (end 110.998 83.312) (width 0.5) (layer "F.Cu") (net 16))
+  (segment (start 109.4232 73.2282) (end 112.29225 73.2282) (width 0.5) (layer "F.Cu") (net 16))
+  (segment (start 108.028 71.833) (end 109.4232 73.2282) (width 0.5) (layer "F.Cu") (net 16))
   (segment (start 108.327 80.772) (end 108.458 80.772) (width 0.5) (layer "F.Cu") (net 16))
-  (segment (start 110.528 71.374) (end 110.528 72.674) (width 0.5) (layer "F.Cu") (net 16))
-  (segment (start 106.807 72.595) (end 108.028 71.374) (width 0.5) (layer "F.Cu") (net 16))
-  (segment (start 113.538 80.772) (end 110.998 83.312) (width 0.5) (layer "F.Cu") (net 16))
+  (segment (start 112.29225 73.2282) (end 113.538 74.47395) (width 0.5) (layer "F.Cu") (net 16))
   (segment (start 128.978 74.994) (end 130.754 76.77) (width 0.5) (layer "B.Cu") (net 16))
   (segment (start 143.764 80.264) (end 142.884 81.144) (width 0.5) (layer "B.Cu") (net 16))
